Commit message: maps | fixed always right turning issue | test files for dc

File: src/waffle/description/lidar.xacro (robot description, xacro)
@@ -1,9 +1,13 @@
 <?xml version="1.0"?>
 <robot xmlns:xacro="http://ros.org/wiki/xacro">
+  <!-- LIDAR properties -->
+  <xacro:property name="lidar_radius" value="0.035"/>  <!-- 35mm -->
+  <xacro:property name="lidar_height" value="0.025"/>  <!-- 25mm -->
+  <xacro:property name="lidar_elevation" value="0.100"/> <!-- 100mm -->
   <!-- LIDAR Definition -->
   <joint name="scan_joint" type="fixed">
     <parent link="base_link"/>
     <child link="laser_frame"/>
-    <origin xyz="-0.064 0 0.122" rpy="0 0 0"/>
+    <origin xyz="0 0 ${lidar_elevation}" rpy="0 0 0"/>
   </joint>
   <link name="laser_frame">
@@ -11,12 +15,12 @@
       <origin xyz="0 0 0" rpy="0 0 0"/>
       <geometry>
-        <cylinder length="0.0315" radius="0.055"/>
+        <cylinder length="${lidar_height}" radius="${lidar_radius}"/>
       </geometry>
       <material name="orange"/>
     </visual>
     <collision>
-      <origin xyz="0.015 0 -0.0065" rpy="0 0 0"/>
+      <origin xyz="0 0 0" rpy="0 0 0"/>
       <geometry>
-        <cylinder length="0.0315" radius="0.055"/>
+        <cylinder length="${lidar_height}" radius="${lidar_radius}"/>
       </geometry>
     </collision>

File: src/waffle/description/waffle_core.xacro (robot description, xacro)
@@ -7,4 +7,13 @@
   <xacro:property name="r200_cam_rgb_pz" value="0.013"/>
   <xacro:property name="r200_cam_depth_offset" value="0.01"/>
+  <!-- Robot dimensions -->
+  <xacro:property name="wheel_radius" value="0.040"/>  <!-- 40mm -->
+  <xacro:property name="wheel_width" value="0.035"/>   <!-- 35mm -->
+  <xacro:property name="wheel_separation" value="0.300"/> <!-- 300mm -->
+  <xacro:property name="wheel_to_front" value="0.060"/> <!-- 60mm -->
+  <xacro:property name="base_width" value="0.265"/>    <!-- 265mm -->
+  <xacro:property name="base_length" value="0.265"/>   <!-- 265mm -->
+  <xacro:property name="base_height" value="0.060"/>   <!-- 60mm -->
+  <xacro:property name="caster_height" value="0.014"/> <!-- 14mm -->
   <!-- Init colour -->
   <material name="black">
@@ -45,18 +54,18 @@
     <parent link="base_footprint"/>
     <child link="base_link" />
-    <origin xyz="0 0 0.010" rpy="0 0 0"/>
+    <origin xyz="0 0 ${wheel_radius + caster_height}" rpy="0 0 0"/>
   </joint>
   <link name="base_link">
     <visual>
-      <origin xyz="0 0 0.047" rpy="0 0 0"/>
-      <geometry>
-        <box size="0.266 0.266 0.094"/>
+      <origin xyz="0 0 ${base_height/2}" rpy="0 0 0"/>
+      <geometry>
+        <box size="${base_length} ${base_width} ${base_height}"/>
       </geometry>
       <material name="red"/>
     </visual>
     <collision>
-      <origin xyz="-0.064 0 0.047" rpy="0 0 0"/>
-      <geometry>
-        <box size="0.266 0.266 0.094"/>
+      <origin xyz="0 0 ${base_height/2}" rpy="0 0 0"/>
+      <geometry>
+        <box size="${base_length} ${base_width} ${base_height}"/>
       </geometry>
     </collision>
@@ -72,5 +81,5 @@
     <parent link="base_link"/>
     <child link="wheel_left_link"/>
-    <origin xyz="0.0 0.144 0.023" rpy="-1.57 0 0"/>
+    <origin xyz="${wheel_to_front} ${wheel_separation/2} 0" rpy="-1.57 0 0"/>
     <axis xyz="0 0 1"/>
   </joint>
@@ -79,5 +88,5 @@
       <origin xyz="0 0 0" rpy="0 0 0"/>
       <geometry>
-        <cylinder length="0.018" radius="0.033"/>
+        <cylinder length="${wheel_width}" radius="${wheel_radius}"/>
       </geometry>
       <material name="blue"/>
@@ -86,5 +95,5 @@
       <origin xyz="0 0 0" rpy="0 0 0"/>
       <geometry>
-        <cylinder length="0.018" radius="0.033"/>
+        <cylinder length="${wheel_width}" radius="${wheel_radius}"/>
       </geometry>
     </collision>
@@ -100,5 +109,5 @@
     <parent link="base_link"/>
     <child link="wheel_right_link"/>
-    <origin xyz="0.0 -0.144 0.023" rpy="-1.57 0 0"/>
+    <origin xyz="${wheel_to_front} -${wheel_separation/2} 0" rpy="-1.57 0 0"/>
     <axis xyz="0 0 1"/>
   </joint>
@@ -107,5 +116,5 @@
       <origin xyz="0 0 0" rpy="0 0 0"/>
       <geometry>
-        <cylinder length="0.018" radius="0.033"/>
+        <cylinder length="${wheel_width}" radius="${wheel_radius}"/>
       </geometry>
       <material name="blue"/>
@@ -114,5 +123,5 @@
       <origin xyz="0 0 0" rpy="0 0 0"/>
       <geometry>
-        <cylinder length="0.018" radius="0.033"/>
+        <cylinder length="${wheel_width}" radius="${wheel_radius}"/>
       </geometry>
     </collision>
@@ -179,90 +188,4 @@
     </inertial>
   </link>
-  <joint name="imu_joint" type="fixed">
-    <parent link="base_link"/>
-    <child link="imu_link"/>
-    <origin xyz="0.0 0 0.068" rpy="0 0 0"/>
-  </joint>
-  <link name="imu_link"/>
-  <joint name="scan_joint" type="fixed">
-    <parent link="base_link"/>
-    <child link="laser_frame"/>
-    <origin xyz="-0.064 0 0.122" rpy="0 0 0"/>
-  </joint>
-  <link name="laser_frame">
-    <visual>
-      <origin xyz="0 0 0" rpy="0 0 0"/>
-      <geometry>
-        <cylinder length="0.0315" radius="0.055"/>
-      </geometry>
-      <material name="orange"/>
-    </visual>
-    <collision>
-      <origin xyz="0.015 0 -0.0065" rpy="0 0 0"/>
-      <geometry>
-        <cylinder length="0.0315" radius="0.055"/>
-      </geometry>
-    </collision>
-    <inertial>
-      <mass value="0.114" />
-      <origin xyz="0 0 0" />
-      <inertia ixx="0.001" ixy="0.0" ixz="0.0"
-               iyy="0.001" iyz="0.0"
-               izz="0.001" />
-    </inertial>
-  </link>
-  <joint name="camera_joint" type="fixed">
-    <origin xyz="0.064 -0.065 0.094" rpy="0 0 0"/>
-    <parent link="base_link"/>
-    <child link="camera_link"/>
-  </joint>
-  <link name="camera_link">
-    <visual>
-      <origin xyz="0 0 0" rpy="1.57 0 1.57"/>
-      <geometry>
-       <mesh filename="package://waffle/description/meshes/sensors/r200.dae" />
-      </geometry>
-    </visual>
-    <collision>
-      <origin xyz="0.003 0.065 0.007" rpy="0 0 0"/>
-      <geometry>
-        <box size="0.012 0.132 0.020"/>
-      </geometry>
-    </collision>
-    <!-- This inertial field needs doesn't contain reliable data!! -->
-    <!--   <inertial>
-          <mass value="0.564" />
-          <origin xyz="0 0 0" />
-          <inertia ixx="0.003881243" ixy="0.0" ixz="0.0"
-                   iyy="0.000498940" iyz="0.0"
-                   izz="0.003879257" />
-        </inertial>-->
-  </link>
-  <joint name="camera_rgb_joint" type="fixed">
-    <origin xyz="0.005 0.018 0.013" rpy="0 0 0"/>
-    <!-- <origin xyz="${r200_cam_rgb_px} ${r200_cam_rgb_py} ${r200_cam_rgb_pz}" rpy="0 0 0"/> -->
-    <parent link="camera_link"/>
-    <child link="camera_rgb_frame"/>
-  </joint>
-  <link name="camera_rgb_frame"/>
-  <joint name="camera_rgb_optical_joint" type="fixed">
-    <origin xyz="0 0 0" rpy="-1.57 0 -1.57"/>
-    <parent link="camera_rgb_frame"/>
-    <child link="camera_rgb_optical_frame"/>
-  </joint>
-  <link name="camera_rgb_optical_frame"/>
-  <joint name="camera_depth_joint" type="fixed">
-    <origin xyz="0.005 0.028 0.013" rpy="0 0 0"/>
-    <!-- <origin xyz="${r200_cam_rgb_px} ${r200_cam_rgb_py + r200_cam_depth_offset} ${r200_cam_rgb_pz}" rpy="0 0 0"/> -->
-    <parent link="camera_link"/>
-    <child link="camera_depth_frame"/>
-  </joint>
-  <link name="camera_depth_frame"/>
-  <joint name="camera_depth_optical_joint" type="fixed">
-    <origin xyz="0 0 0" rpy="-1.57 0 -1.57"/>
-    <parent link="camera_depth_frame"/>
-    <child link="camera_depth_optical_frame"/>
-  </joint>
-  <link name="camera_depth_optical_frame"/>
   <!-- Gazebo materials -->
   <gazebo reference="base_link">
@@ -398,6 +321,6 @@
       <left_joint>wheel_left_joint</left_joint>
       <right_joint>wheel_right_joint</right_joint>
-      <wheel_separation>0.288</wheel_separation>
-      <wheel_diameter>0.066</wheel_diameter>
+      <wheel_separation>${wheel_separation}</wheel_separation>
+      <wheel_diameter>${wheel_radius * 2}</wheel_diameter>
       <max_wheel_torque>20</max_wheel_torque>
       <max_wheel_acceleration>1.0</max_wheel_acceleration>
